File: halfVoltageMosfetBoard.kicad_pcb (KiCad board)
At the start: 2 copper layers, 76 x 58.2 mm, 49 parts, among them J1 Phoenix 1987740, J2 Phoenix 1987740, J5 Phoenix 1729018, Q1 Q_NMOS_DGS, Q2 Q_NMOS_DGS, U1 STM32L011F3Px, U2 MCP1703A-3302_SOT89, U3 XC6702-3.3, U4 MIC4126

Commit message: Revision 2 changes see readme Added text to readme Exported schematic
Parts:
- added D4: BZX84C3V3 3.3V, Diode_SMD:D_SOT-23_ANK, F.Cu at (146.0, 94.8)
- added D5: BZX84C3V3 3.3V, Diode_SMD:D_SOT-23_ANK, F.Cu at (145.2, 99.8)
- R1, R3: value 100k -> 20k
- moved C4 9.95 mm to (143.0, 94.8)
- moved C5 9.78 mm to (142.8, 104.5)
- moved R2 1.75 mm to (141.0, 104.5)
- turned R4 to 270 degrees
Connections:
- C4 pad 1: /InputHeater1 -> /InputHeater2
- C5 pad 1: /InputHeater2 -> /InputHeater1
- J5 pad 1: /InputHeater2 -> Net-(J5-Pad1)
- J5 pad 2: /InputHeater1 -> Net-(J5-Pad2)
- R1 pad 2: /InputHeater1 -> Net-(J5-Pad2)
- R2 pad 1: /InputHeater1 -> Net-(J5-Pad2)
- R2 pad 2: GND -> /InputHeater1
- R3 pad 2: /InputHeater2 -> Net-(J5-Pad1)
- R4 pad 2: GND -> Net-(J5-Pad1)
Routing:
- net /InputHeater2: track 30.1 -> 22.1 mm
- net Net-(J5-Pad2): track 0.00 -> 7.42 mm
- net Net-(J5-Pad1): track 0.00 -> 7.38 mm
- net /InputHeater1: track 33.1 -> 27.4 mm
- net GND: track 87.9 -> 92.7 mm
Other:
- board text added: "M.A. 2021 Drives 12V Heaters with 24V input Rev 2 Heater 1 - Bed Heater 2 - Extruder"
- board text removed: "M.A. 2021 Drives 12V Heaters with 24V input Rev 1 Heater 1 - Bed Heater 2 - Extruder"
