File: halfVoltageMosfetBoard.sch (KiCad schematic (older format))
At the start: 49 parts, among them J1 Phoenix 1987740, J2 Phoenix 1987740, J5 Phoenix 1729018, Q1 Q_NMOS_DGS, Q2 Q_NMOS_DGS, U1 STM32L011F3Px, U2 MCP1703A-3302_SOT89, U3 XC6702-3.3, U4 MIC4126

Commit message: finished layout rev A
Connections:
- net EnableHeater1 is gone; now on net InputHeater1: C4.1, J5.2 (Pin_2), R1.2, R2.1
- net EnableHeater2 is gone; now on net InputHeater2: C5.1, J5.1 (Pin_1), R3.2, R4.1
- net +3V3: now also U1.13 (PA7)
- net GND: now also R12.1; no longer R12.2
- net Heater1: now also R9.2, U4.4 (InB); no longer R8.2, U4.2 (InA)
- net Heater1ActiveLed: now also U1.14 (PB1)
- net Heater2: now also R8.2, U4.2 (InA); no longer R9.2, U4.4 (InB)
- net Heater2ActiveLed: now also U1.10 (PA4)
- net Temp: now also U1.12 (PA6); no longer U1.6 (PA0)
- net at R10.2, U4.5 (OutB): now also R12.2
- net at R11.1, U4.7 (OutA): now also R13.1
- net at Q1.2 (G), R10.1: no longer R12.1
- net at Q2.2 (G), R11.2: no longer R13.1
- net InputHeater2: now reaches U1.7 (PA1)
- net InputHeater1: now reaches U1.9 (PA3)
- net Stage1 renamed PowerHeater1
- net PowerHeater1: now also J2.4 (Pin_4); no longer J2.3 (Pin_3)
- net Stage2 renamed PowerHeater2
- net PowerHeater2: now also J2.3 (Pin_3); no longer J2.4 (Pin_4)
- no-connect marks 14 -> 7
Other:
- note removed: "5V compatible gpio"
- moved on the sheet: R12, R13
Changed lines of the file:
@@
 L Device:R R12
 U 1 1 6099C86E
-P 8600 1250
-F 0 "R12" H 8670 1296 50  0000 L CNN
-F 1 "100k" H 8670 1205 50  0000 L CNN
-F 2 "Resistor_SMD:R_0603_1608Metric" V 8530 1250 50  0001 C CNN
-F 3 "~" H 8600 1250 50  0001 C CNN
-	1    8600 1250
+P 7750 850
+F 0 "R12" H 7820 896 50  0000 L CNN
+F 1 "100k" H 7820 805 50  0000 L CNN
+F 2 "Resistor_SMD:R_0603_1608Metric" V 7680 850 50  0001 C CNN
+F 3 "~" H 7750 850 50  0001 C CNN
+	1    7750 850
 	1    0    0    -1
 $EndComp
@@
 	1    0    0    -1
 $EndComp
-Wire Wire Line
-	8700 1050 8600 1050
-Wire Wire Line
-	8600 1100 8600 1050
-Wire Wire Line
-	8600 1400 8600 1450
-Wire Wire Line
-	8600 1450 9000 1450
 $Comp
 L power:GND #PWR0105
@@
 	1    0    0    -1
 $EndComp
-Wire Wire Line
-	9000 1500 9000 1450
-Connection ~ 9000 1450
 $Comp
 L Device:R R13
 U 1 1 609AD4E5
-P 8600 2250
-F 0 "R13" H 8670 2296 50  0000 L CNN
-F 1 "100k" H 8670 2205 50  0000 L CNN
-F 2 "Resistor_SMD:R_0603_1608Metric" V 8530 2250 50  0001 C CNN
-F 3 "~" H 8600 2250 50  0001 C CNN
-	1    8600 2250
+P 7750 1900
+F 0 "R13" H 7820 1946 50  0000 L CNN
+F 1 "100k" H 7820 1855 50  0000 L CNN
+F 2 "Resistor_SMD:R_0603_1608Metric" V 7680 1900 50  0001 C CNN
+F 3 "~" H 7750 1900 50  0001 C CNN
+	1    7750 1900
 	1    0    0    -1
 $EndComp
@@
 	1    0    0    -1
 $EndComp
-Wire Wire Line
-	8700 2050 8600 2050
-Wire Wire Line
-	8600 2100 8600 2050
-Wire Wire Line
-	8600 2400 8600 2450
-Wire Wire Line
-	8600 2450 9000 2450
 $Comp
 L power:GND #PWR0106
@@
 	1    0    0    -1
 $EndComp
-Wire Wire Line
-	9000 2500 9000 2450
-Connection ~ 9000 2450
 Wire Wire Line
 	9000 850  9000 800
@@
 Wire Wire Line
 	10750 1650 10750 1700
-Wire Wire Line
-	9000 1250 9000 1450
-Wire Wire Line
-	9000 2250 9000 2450
 $Comp
 L Device:C C13
@@
 close to mic4126
 $Comp
-L MIC4126:MIC4126 U4
-U 1 1 6099B1A3
-P 7250 750
-F 0 "U4" H 7500 350 50  0000 C CNN
-F 1 "MIC4126" H 7500 250 50  0000 C CNN
-F 2 "Package_SO:SOIC-8-1EP_3.9x4.9mm_P1.27mm_EP2.29x3mm_ThermalVias" H 7550 400 50  0001 C CNN
-F 3 "" H 7550 400 50  0001 C CNN
-	1    7250 750
-	1    0    0    -1
-$EndComp
-$Comp
 L Device:CP C18
 U 1 1 609E1535
@@
 	9500 3550 9500 3500
 Wire Wire Line
-	7650 1600 8100 1600
+	7650 1600 7750 1600
 $Comp
 L Device:CP C17
@@
 	9150 3500 9500 3500
 Wire Wire Line
-	8100 1500 7650 1500
+	8100 1500 7750 1500
 Wire Wire Line
 	8450 3500 8800 3500
@@
 Text Label 3650 7050 0    50   ~ 0
 Temp
+Text Label 6250 1600 2    50   ~ 0
+Heater1
 Text Label 6250 1500 2    50   ~ 0
-Heater1
-Text Label 6250 1600 2    50   ~ 0
 Heater2
 $Comp
@@
 Wire Wire Line
 	1700 3300 1750 3300
-Text Label 2200 3550 0    50   ~ 0
+Text Label 2200 4150 0    50   ~ 0
 Temp
-Wire Wire Line
-	2200 3550 2150 3550
 Text Label 2200 3750 0    50   ~ 0
 Heater1
@@
 Text Notes 600  7650 0    50   ~ 10
 Connect these to the !negative! \nTerminal of your 24V Motherboards \npower output
-Text Label 5800 5300 2    50   ~ 0
+Text Label 2200 3950 0    50   ~ 0
 Heater2ActiveLed
-Text Label 5800 5200 2    50   ~ 0
+Text Label 1200 4550 2    50   ~ 0
 Heater1ActiveLed
-Text Label 2450 6350 0    50   ~ 0
-EnableHeater1
-Text Label 2450 6450 0    50   ~ 0
-EnableHeater2
-Text Label 5800 5100 2    50   ~ 0
-EnableHeater1
-Text Label 5800 5000 2    50   ~ 0
-EnableHeater2
 Text Notes 600  5500 0    50   ~ 10
 Heater Command input
@@
 Wire Wire Line
 	10350 2600 10350 2550
+Text Label 10350 2850 2    50   ~ 0
+PowerHeater1
+Wire Wire Line
+	10350 2750 10400 2750
 Text Label 10350 2750 2    50   ~ 0
-Stage1
-Wire Wire Line
-	10350 2750 10400 2750
-Text Label 10350 2850 2    50   ~ 0
-Stage2
+PowerHeater2
 Wire Wire Line
 	10350 2850 10400 2850
@@
 Wire Wire Line
 	8100 1100 8100 1050
-Wire Wire Line
-	8100 1050 8600 1050
-Connection ~ 8600 1050
-Wire Wire Line
-	8100 2050 8600 2050
-Connection ~ 8600 2050
 Text Label 9200 800  0    50   ~ 0
-Stage1
+PowerHeater1
 Text Label 9200 1800 0    50   ~ 0
-Stage2
+PowerHeater2
 Wire Wire Line
 	9000 1800 9200 1800
@@
 	9200 800  9000 800
 Text Label 10500 1200 2    50   ~ 0
-Stage1
+PowerHeater1
 Wire Wire Line
 	10550 1200 10550 1300
 Text Label 10500 2100 2    50   ~ 0
-Stage2
+PowerHeater2
 Wire Wire Line
 	10550 2000 10550 2100
@@
 Wire Notes Line
 	11150 4200 11150 550
-NoConn ~ 5800 5300
-NoConn ~ 5800 5200
 NoConn ~ 1250 4650
-NoConn ~ 1250 4550
 NoConn ~ 1250 4350
 NoConn ~ 1250 4250
 NoConn ~ 2150 4450
 NoConn ~ 2150 4350
-NoConn ~ 2150 4250
-NoConn ~ 2150 4150
-NoConn ~ 2150 3850
-NoConn ~ 2150 3950
-NoConn ~ 2150 3650
-Text Notes 5800 5000 0    50   ~ 10
-5V compatible gpio
-Text Notes 5800 5100 0    50   ~ 10
-5V compatible gpio
 $Comp
 L Mechanical:MountingHole H1
@@
 	1    0    0    -1
 $EndComp
+Wire Wire Line
+	8100 2050 8700 2050
+$Comp
+L MIC4126:MIC4126 U4
+U 1 1 6099B1A3
+P 7250 750
+F 0 "U4" H 7500 350 50  0000 C CNN
+F 1 "MIC4126" H 7500 250 50  0000 C CNN
+F 2 "Package_SO:SOIC-8-1EP_3.9x4.9mm_P1.27mm_EP2.29x3mm_ThermalVias" H 7550 400 50  0001 C CNN
+F 3 "" H 7550 400 50  0001 C CNN
+	1    7250 750
+	1    0    0    -1
+$EndComp
+$Comp
+L power:GND #PWR0107
+U 1 1 611A554B
+P 7750 2100
+F 0 "#PWR0107" H 7750 1850 50  0001 C CNN
+F 1 "GND" H 7755 1927 50  0000 C CNN
+F 2 "" H 7750 2100 50  0001 C CNN
+F 3 "" H 7750 2100 50  0001 C CNN
+	1    7750 2100
+	1    0    0    -1
+$EndComp
+Wire Wire Line
+	7750 2050 7750 2100
+Wire Wire Line
+	9000 2250 9000 2500
+Wire Wire Line
+	8100 1050 8700 1050
+Wire Wire Line
+	9000 1250 9000 1500
+$Comp
+L power:GND #PWR0144
+U 1 1 611B8FDB
+P 7550 700
+F 0 "#PWR0144" H 7550 450 50  0001 C CNN
+F 1 "GND" H 7555 527 50  0000 C CNN
+F 2 "" H 7550 700 50  0001 C CNN
+F 3 "" H 7550 700 50  0001 C CNN
+	1    7550 700
+	1    0    0    -1
+$EndComp
+Wire Wire Line
+	7750 700  7750 650
+Wire Wire Line
+	7750 650  7550 650
+Wire Wire Line
+	7550 650  7550 700
+Wire Wire Line
+	7750 1750 7750 1600
+Connection ~ 7750 1600
+Wire Wire Line
+	7750 1600 8100 1600
+Wire Wire Line
+	7750 1500 7750 1000
+Connection ~ 7750 1500
+Wire Wire Line
+	7750 1500 7650 1500
+Wire Wire Line
+	2150 4150 2200 4150
+NoConn ~ 2150 3550
+Text Label 2200 3850 0    50   ~ 0
+InputHeater1
+Text Label 2200 3650 0    50   ~ 0
+InputHeater2
+Wire Wire Line
+	2200 3850 2150 3850
+Wire Wire Line
+	2200 3650 2150 3650
+Wire Wire Line
+	2150 4250 2900 4250
+Wire Wire Line
+	2900 4250 2900 4150
+$Comp
+L power:+3V3 #PWR0145
+U 1 1 61329EA7
+P 2900 4150
+F 0 "#PWR0145" H 2900 4000 50  0001 C CNN
+F 1 "+3V3" H 2915 4323 50  0000 C CNN
+F 2 "" H 2900 4150 50  0001 C CNN
+F 3 "" H 2900 4150 50  0001 C CNN
+	1    2900 4150
+	1    0    0    -1
+$EndComp
+Wire Wire Line
+	1200 4550 1250 4550
+Wire Wire Line
+	2200 3950 2150 3950
+Text Label 2450 6450 0    50   ~ 0
+InputHeater2
+Text Label 2450 6350 0    50   ~ 0
+InputHeater1
 $EndSCHEMATC
